File: com-express-7-baseboard.kicad_pcb (KiCad board)
At the start: 2 copper layers, 225 x 110.2 mm, 14 parts, among them J9 Edge_Conn_Bus_PCIe_x4

Commit message: [#56643] Add necessary blocks to schematic
Parts:
- REF**: footprint antmicro-footprints:LX2160A-CEX7 -> com-express-7-baseboard-footprints:LX2160A-CEX7
- REF**: footprint antmicro-footprints:SFP_SS-79100-010 -> com-express-7-baseboard-footprints:SFP_SS-79100-010
- REF**: footprint antmicro-footprints:RJ45_RJE361882415 -> com-express-7-baseboard-footprints:RJ45_RJE361882415
- REF** (x2): footprint antmicro-footprints:Mech_M2_2280_H2.5mm -> com-express-7-baseboard-footprints:Mech_M2_2280_H2.5mm
- REF**: footprint antmicro-footprints:Bus_M.2_Socket_Key_E_TE_2199230-4 -> com-express-7-baseboard-footprints:Bus_M.2_Socket_Key_E_TE_2199230-4
- REF**: footprint antmicro-footprints:USB-C_Receptacle_WE_632723300011 -> com-express-7-baseboard-footprints:USB-C_Receptacle_WE_632723300011
- REF**: footprint antmicro-footprints:RJ45_RJE1R288335413 -> com-express-7-baseboard-footprints:RJ45_RJE1R288335413
- REF**: footprint antmicro-footprints:Molex_Mini-Fit_2x4_172448-0008_Horizontal -> com-express-7-baseboard-footprints:Molex_Mini-Fit_2x4_172448-0008_Horizontal
- REF**: footprint antmicro-footprints:Mech_M2_2230_H2.5mm -> com-express-7-baseboard-footprints:Mech_M2_2230_H2.5mm
- REF**: footprint antmicro-footprints:HDMI-A_Receptacle_TE_2007435-1 -> com-express-7-baseboard-footprints:HDMI-A_Receptacle_TE_2007435-1
