File: misc.kicad_sch (KiCad schematic)
At the start: 51 parts, among them J10 Molex_KK_1x4_0470531000, J8 Molex_KK_1x4_0470531000, J9 Molex_KK_1x4_0470531000, Q1 MMBT3904LT1G, Q10 BSS138PW, Q11 PJE138K, Q12 PJE138K, Q2 MMBT3904LT1G, Q9 BSS84AKW, U18 ADT7476AARQZ, U19 74LVC1G157-Q100H_SOT457, U20 74LVC1G157-Q100H_SOT457, U21 NTS0102_TSSOP, U22 NTS0102_TSSOP, U23 NTS0102_TSSOP

Commit message: Fix ERC
Parts:
- added R323, R324: R_10k_0402, antmicro-footprints:R_0402_1005Metric, symbol antmicroResistors0402:R_10k_0402
Connections:
- net +3V3: now also R323.2, R324.2
- net PWM1: now also R323.1
- net PWM2: now also R324.1
Other:
- moved on the sheet: R117
